File: kicad/z2_interface.kicad_sch (KiCad schematic)
At the start: 34 parts

Commit message: eda: aplicar footprints verificados y regenerar hierarchy PR15
Parts:
- U_HMI_LVL: footprint Package_MSOP:VSSOP-8_2x3.1mm_P0.65mm -> NFB:TI_DCU0008A_TXU0202
Changed lines of the file:
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@@
     (property "Reference" "U_HMI_LVL" (at 347.98 78.74 0) (effects (font (size 1 1))))
     (property "Value" "TXU0202" (at 347.98 81.28 0) (effects (font (size 0.9 0.9))))
-    (property "Footprint" "Package_MSOP:VSSOP-8_2x3.1mm_P0.65mm" (at 347.98 83.82 0) (effects (font (size 0.8 0.8)) (hide yes)))
+    (property "Footprint" "NFB:TI_DCU0008A_TXU0202" (at 347.98 83.82 0) (effects (font (size 0.8 0.8)) (hide yes)))
     (property "Datasheet" "~" (at 347.98 81.28 0) (effects (font (size 0.8 0.8)) (hide yes)))
     (property "MPN" "TXU0202DCUR" (at 347.98 86.36 0) (effects (font (size 0.8 0.8)) (hide yes)))
