File: kicad/z4_interface.kicad_sch (KiCad schematic)
At the start: 31 parts

Commit message: eda: aplicar footprints verificados y regenerar hierarchy PR15
Parts:
- J_CHILLER_CTL, J_CO2_SOL, J_PUMP: footprint TerminalBlock_Phoenix:PhoenixContact_MSTBA-G_02x5.08mm_Angled -> Connector_Phoenix_MSTB:PhoenixContact_MSTBA_2,5_2-G-5,08_1x02_P5.08mm_Horizontal
Changed lines of the file:
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@@
     (property "Reference" "J_PUMP" (at 289.56 78.74 0) (effects (font (size 1 1))))
     (property "Value" "MSTBA 2,5/2-G-5,08" (at 289.56 81.28 0) (effects (font (size 0.9 0.9))))
-    (property "Footprint" "TerminalBlock_Phoenix:PhoenixContact_MSTBA-G_02x5.08mm_Angled" (at 289.56 83.82 0) (effects (font (size 0.8 0.8)) (hide yes)))
+    (property "Footprint" "Connector_Phoenix_MSTB:PhoenixContact_MSTBA_2,5_2-G-5,08_1x02_P5.08mm_Horizontal" (at 289.56 83.82 0) (effects (font (size 0.8 0.8)) (hide yes)))
     (property "Datasheet" "~" (at 289.56 81.28 0) (effects (font (size 0.8 0.8)) (hide yes)))
     (property "MPN" "1757242" (at 289.56 86.36 0) (effects (font (size 0.8 0.8)) (hide yes)))
@@
     (property "Reference" "J_CO2_SOL" (at 231.14 170.18 0) (effects (font (size 1 1))))
     (property "Value" "MSTBA 2,5/2-G-5,08" (at 231.14 172.72 0) (effects (font (size 0.9 0.9))))
-    (property "Footprint" "TerminalBlock_Phoenix:PhoenixContact_MSTBA-G_02x5.08mm_Angled" (at 231.14 175.26 0) (effects (font (size 0.8 0.8)) (hide yes)))
+    (property "Footprint" "Connector_Phoenix_MSTB:PhoenixContact_MSTBA_2,5_2-G-5,08_1x02_P5.08mm_Horizontal" (at 231.14 175.26 0) (effects (font (size 0.8 0.8)) (hide yes)))
     (property "Datasheet" "~" (at 231.14 172.72 0) (effects (font (size 0.8 0.8)) (hide yes)))
     (property "MPN" "1757242" (at 231.14 177.8 0) (effects (font (size 0.8 0.8)) (hide yes)))
@@
     (property "Reference" "J_CHILLER_CTL" (at 289.56 215.9 0) (effects (font (size 1 1))))
     (property "Value" "MSTBA 2,5/2-G-5.08" (at 289.56 218.44 0) (effects (font (size 0.9 0.9))))
-    (property "Footprint" "TerminalBlock_Phoenix:PhoenixContact_MSTBA-G_02x5.08mm_Angled" (at 289.56 220.98 0) (effects (font (size 0.8 0.8)) (hide yes)))
+    (property "Footprint" "Connector_Phoenix_MSTB:PhoenixContact_MSTBA_2,5_2-G-5,08_1x02_P5.08mm_Horizontal" (at 289.56 220.98 0) (effects (font (size 0.8 0.8)) (hide yes)))
     (property "Datasheet" "~" (at 289.56 218.44 0) (effects (font (size 0.8 0.8)) (hide yes)))
     (property "MPN" "1757242" (at 289.56 223.52 0) (effects (font (size 0.8 0.8)) (hide yes)))
