File: kicad/z3_interface.kicad_sch (KiCad schematic)
At the start: 34 parts

Commit message: eda: aplicar footprints verificados y regenerar hierarchy PR15
Parts:
- J_PWR_IN: footprint TerminalBlock_Phoenix:PhoenixContact_MSTBA-G_02x5.08mm_Angled -> Connector_Phoenix_MSTB:PhoenixContact_MSTBA_2,5_2-G-5,08_1x02_P5.08mm_Horizontal
Changed lines of the file:
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@@
     (property "Reference" "J_PWR_IN" (at 55.88 33.02 0) (effects (font (size 1 1))))
     (property "Value" "MSTBA 2,5/2-G-5,08" (at 55.88 35.56 0) (effects (font (size 0.9 0.9))))
-    (property "Footprint" "TerminalBlock_Phoenix:PhoenixContact_MSTBA-G_02x5.08mm_Angled" (at 55.88 38.1 0) (effects (font (size 0.8 0.8)) (hide yes)))
+    (property "Footprint" "Connector_Phoenix_MSTB:PhoenixContact_MSTBA_2,5_2-G-5,08_1x02_P5.08mm_Horizontal" (at 55.88 38.1 0) (effects (font (size 0.8 0.8)) (hide yes)))
     (property "Datasheet" "~" (at 55.88 35.56 0) (effects (font (size 0.8 0.8)) (hide yes)))
     (property "MPN" "1757242" (at 55.88 40.64 0) (effects (font (size 0.8 0.8)) (hide yes)))

Commit message: eda: aplicar footprints verificados y regenerar hierarchy PR15
Parts:
- F_ACT: footprint Fuse:Fuse_2410_6125Metric -> NFB:Littelfuse_0454_NANO2
Changed lines of the file:
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@@
     (property "Reference" "F_ACT" (at 114.3 124.46 0) (effects (font (size 1 1))))
     (property "Value" "1.5A 125V Slo-Blo Nano2" (at 114.3 127 0) (effects (font (size 0.9 0.9))))
-    (property "Footprint" "Fuse:Fuse_2410_6125Metric" (at 114.3 129.54 0) (effects (font (size 0.8 0.8)) (hide yes)))
+    (property "Footprint" "NFB:Littelfuse_0454_NANO2" (at 114.3 129.54 0) (effects (font (size 0.8 0.8)) (hide yes)))
     (property "Datasheet" "~" (at 114.3 127 0) (effects (font (size 0.8 0.8)) (hide yes)))
     (property "MPN" "045401.5MR" (at 114.3 132.08 0) (effects (font (size 0.8 0.8)) (hide yes)))
