File: kicad/NFB_Insight_PCBA_v2.kicad_pcb (KiCad board)
At the start: 4 copper layers, 242.3 x 68.6 mm, 120 parts

Commit message: placement: acercar testpoints load-cell al HX711 antes de routing
ECO localizado Z2 previo a routing.

- mueve únicamente TP_LOAD_A_POS y TP_LOAD_A_NEG cerca de U_HX;
- conserva el ECO PR22 Z3 del TPSM33625;
- valida 2 refs movidas / 117 intactas;
- mantiene outline, zonas, netlist, footprints y routing sin cambios;
- DRC físico: 0 errores, sin shorts/clearance/courtyard;
- deuda placement-only: 255 warnings silk/text acotados, 4 menos que PR22, y 250 unconnected;
- hace composicional el gate histórico PR22: valida su delta local contra PR17 y reproduce la cadena ECO vigente antes de manifest/PCB/DRC.

PR24 no agrega routing. El siguiente checkpoint reinicia PR19A limpio con política 28/28 o no merge.
Parts:
- moved TP_LOAD_A_NEG 35.5 mm to (112.8, 29.3)
- moved TP_LOAD_A_POS 35.3 mm to (110.2, 29.3)

Commit message: routing: cerrar PR19A 28/28 nets locales
Cierra el primer lote físico de routing PR19A sobre el baseline post-PR24/PR25.

- 28/28 nets locales con cobre.
- 31/31 nets futuras intactas.
- 523 segmentos y 24 vías.
- In1.Cu sin signal routing; 0 copper zones.
- KiCad 10.0.5 DRC: 0 errors.
- 255 warnings conocidos exclusivamente de serigrafía/texto.
- 204 unconnected restantes, ninguno perteneciente a PR19A.
- 5V_PGOOD simplificado de 143 a 12 segmentos.
- WDT_MR_N simplificado de 100 a 10 segmentos.
- Gates históricos adaptados de forma composicional sin relajar contratos.
- README.md actualizado con el checkpoint y PR19B como siguiente lote.
Routing:
- net 5V_PGOOD: track 0.00 -> 68.9 mm
- net CO2_OPENLOAD_N: track 0.00 -> 54.2 mm, vias 0 -> 4
- net LOAD_A_POS: track 0.00 -> 51.9 mm, vias 0 -> 1
- net LOAD_A_NEG: track 0.00 -> 51.4 mm, vias 0 -> 2
- net WDT_MR_N: track 0.00 -> 47.7 mm
- net HMI_FIELD_TX: track 0.00 -> 30.6 mm, vias 0 -> 1
- net CO2_EN_DRV: track 0.00 -> 30.3 mm, vias 0 -> 2
- net HX_VBG: track 0.00 -> 25.6 mm
- net PUMP_SR_CFG: track 0.00 -> 24.2 mm, vias 0 -> 2
- net HMI_FIELD_RX: track 0.00 -> 24.1 mm
- net PH_FIELD_SIG: track 0.00 -> 22.6 mm
- net DO_FIELD_SIG: track 0.00 -> 21.6 mm
- net ORP_FIELD_SIG: track 0.00 -> 21.2 mm
- net CHILLER_CONTACT_B: track 0.00 -> 20.2 mm
- net CHILLER_CONTACT_A: track 0.00 -> 19.9 mm
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