File: kicad/NFB_Insight_PCBA_v2.kicad_pcb (KiCad board)
At the start: 4 copper layers, 242.3 x 68.6 mm, 120 parts

Commit message: routing: persistir PR19B 4/4 con DRC 0
Routing:
- net PUMP_CURRENT_ADC: track 0.00 -> 232.5 mm, vias 0 -> 4
- net DO_ADC: track 0.00 -> 105.4 mm, vias 0 -> 1
- net ORP_ADC: track 0.00 -> 77.1 mm, vias 0 -> 1
- net PH_ADC: track 0.00 -> 47.2 mm, vias 0 -> 1

Commit message: routing: persistir checkpoint PR19C 16/16 DRC=0
Routing:
- net ACT_FAULT_N: track 0.00 -> 397.7 mm, vias 0 -> 8
- net CHILLER_CTL: track 0.00 -> 296.2 mm, vias 0 -> 4
- net CO2_SOL_CTL: track 0.00 -> 278.9 mm, vias 0 -> 8
- net PUMP_DIR: track 0.00 -> 276.9 mm, vias 0 -> 8
- net PUMP_PWM: track 0.00 -> 265.4 mm, vias 0 -> 4
- net I2C_SCL: track 0.00 -> 260.0 mm, vias 0 -> 9
- net I2C_SDA: track 0.00 -> 250.6 mm, vias 0 -> 9
- net HMI_TX: track 0.00 -> 227.9 mm, vias 0 -> 8
- net HMI_RX: track 0.00 -> 225.6 mm, vias 0 -> 9
- net HX711_SCK: track 0.00 -> 195.1 mm, vias 0 -> 5
- net HX711_DOUT: track 0.00 -> 181.7 mm, vias 0 -> 2
- net MCU_WDI: track 0.00 -> 180.3 mm, vias 0 -> 3
- net LED_STATUS: track 0.00 -> 177.3 mm, vias 0 -> 4
- net UNO_IOREF_3V3: track 0.00 -> 156.4 mm, vias 0 -> 2
- net MCU_NRST: track 0.00 -> 121.9 mm, vias 0 -> 3
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
Commit message: power: cerrar ECO HMI con 5V_HMI dedicado y PR19D
Connections:
- C_HMI_B pad 1: 5V_RAIL -> 5V_HMI
- J_HMI pad 1: 5V_RAIL -> 5V_HMI
- U_HMI_LVL pad 7: 5V_RAIL -> 5V_HMI
Routing:
- net 5V_HMI: track 0.00 -> 36.4 mm, vias 0 -> 2
Changed lines of the file:
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@@
 			(layers "F.Cu" "F.Mask" "F.Paste")
 			(roundrect_rratio 0.166667)
-			(net "5V_RAIL")
+			(net "5V_HMI")
 		)
 		(pad "8" smd roundrect
@@
 			(remove_unused_layers no)
 			(roundrect_rratio 0.147059)
-			(net "5V_RAIL")
+			(net "5V_HMI")
 		)
 		(pad "2" thru_hole oval
@@
 			(layers "F.Cu" "F.Mask" "F.Paste")
 			(roundrect_rratio 0.25)
-			(net "5V_RAIL")
+			(net "5V_HMI")
 		)
 		(pad "2" smd roundrect
@@
 		(net "LED_STATUS")
 	)
+	(segment
+		(start 148.815 20.835)
+		(end 148.815 22.2)
+		(width 0.4)
+		(layer "F.Cu")
+		(net "5V_HMI")
+	)
+	(segment
+		(start 157.035 17.775)
+		(end 158.2 17.775)
+		(width 0.2)
+		(layer "F.Cu")
+		(net "5V_HMI")
+	)
+	(via
+		(at 158.2 17.775)
+		(size 0.8)
+		(drill 0.4)
+		(layers "F.Cu" "B.Cu")
+		(net "5V_HMI")
+	)
+	(via
+		(at 148.815 22.2)
+		(size 0.8)
+		(drill 0.4)
+		(layers "F.Cu" "B.Cu")
+		(net "5V_HMI")
+	)
+	(segment
+		(start 150 22.2)
+		(end 148.815 22.2)
+		(width 0.4)
+		(layer "In2.Cu")
+		(net "5V_HMI")
+	)
+	(segment
+		(start 158.2 12)
+		(end 158.2 17.775)
+		(width 0.4)
+		(layer "In2.Cu")
+		(net "5V_HMI")
+	)
+	(segment
+		(start 151.635 3.635)
+		(end 150 12)
+		(width 0.4)
+		(layer "In2.Cu")
+		(net "5V_HMI")
+	)
+	(segment
+		(start 150 12)
+		(end 150 22.2)
+		(width 0.4)
+		(layer "In2.Cu")
+		(net "5V_HMI")
+	)
+	(segment
+		(start 150 12)
+		(end 158.2 12)
+		(width 0.4)
+		(layer "In2.Cu")
+		(net "5V_HMI")
+	)
 	(embedded_fonts no)
